Commit message: Added Central Laser

File: prius_description/urdf/prius.urdf (robot description, URDF)
Before this commit: robot prius, 25 links, 24 joints
Links:
- added link main_laser_link, mass 1
Joints:
- added joint main_laser_joint: type fixed, parent chassis, child main_laser_link, origin xyz=0.0 -2.3 0.5 rpy=0 0 0
